File: PCB/DronDozator/DronDozator.kicad_sch (KiCad schematic)
At the start: 7 parts, among them U1 LM2596

Commit message: Finalized schem
Parts:
- added An1, An2, An3: Conn_01x03_Socket, Connector_PinSocket_2.54mm:PinSocket_1x03_P2.54mm_Vertical, symbol Connector:Conn_01x03_Socket
- added C1: 100uF, Capacitor_THT:CP_Radial_D6.3mm_P2.50mm, symbol Device:C_Polarized
- added D1: LED, LED_THT:LED_D4.0mm, symbol Device:LED
- added H1, H2, H3, H4: MountingHole_Pad, MountingHole:MountingHole_3.5mm_Pad, symbol Mechanical:MountingHole_Pad
- added R1, R2, R3: 10k, Resistor_THT:R_Axial_DIN0204_L3.6mm_D1.6mm_P7.62mm_Horizontal, symbol Device:R
- added SW1, SW2, SW3: SW_Push, Button_Switch_THT:SW_PUSH_6mm, symbol Switch:SW_Push
- added UART1, UART2: Conn_01x04_Socket, Connector_PinSocket_2.54mm:PinSocket_1x04_P2.54mm_Vertical, symbol Connector:Conn_01x04_Socket
- Motor1: footprint Connector_PinSocket_2.54mm:PinSocket_1x04_P2.54mm_Vertical -> Connector_PinHeader_2.54mm:PinHeader_1x04_P2.54mm_Vertical
- renumbered U1 to Converter1
Connections:
- net GND: now reaches Power1.1 (Pin_1)
- net GND: now also Arduino1.29 (GND), Arduino1.4 (GND), Converter1.2 (IN-), Converter1.4 (OUT-), Display1.1 (Pin_1), Driver1.1 (GND), Driver1.10 (MS1), Driver1.12 (MS3), Driver1.7 (GND), Driver1.9 (~{ENABLE}), GPS1.4 (Pin_4), An1.3 (Pin_3), An2.3 (Pin_3), An3.3 (Pin_3), C1.2, D1.1 (K), H1.1, H2.1, H3.1, H4.1, SW1.2, SW2.2, SW3.2, UART1.4 (Pin_4), UART2.4 (Pin_4)
- net VCC: now reaches Power1.2 (Pin_2)
- net VCC: now also Converter1.1 (IN+), Driver1.8 (VMOT), C1.1
- net +5V: now reaches Driver1.11 (MS2)
- net +5V: now also Arduino1.27 (+5V), Converter1.3 (OUT+), Display1.2 (Pin_2), Driver1.2 (VDD), GPS1.1 (Pin_1), An1.1 (Pin_1), An2.1 (Pin_1), An3.1 (Pin_1), R1.1, R2.1, R3.1, UART1.1 (Pin_1), UART2.1 (Pin_1)
- net at Driver1.13 (~{RESET}): now also Driver1.14 (~{SLEEP})
- net STEP: now reaches Driver1.15 (STEP)
- net STEP: now also Arduino1.10 (D7)
- net DIR: now reaches Driver1.16 (DIR)
- net DIR: now also Arduino1.9 (D6)
- net at Driver1.3 (1B): now also Motor1.4 (Pin_4)
- net at Driver1.4 (1A): now also Motor1.3 (Pin_3)
- net at Driver1.5 (2A): now also Motor1.2 (Pin_2)
- net at Driver1.6 (2B): now also Motor1.1 (Pin_1)
- net CS: now reaches Arduino1.11 (D8)
- net CS: now also Display1.7 (Pin_7)
- net RES: now reaches Arduino1.12 (D9)
- net RES: now also Display1.5 (Pin_5)
- net DC: now reaches Arduino1.13 (D10)
- net DC: now also Display1.6 (Pin_6)
- net MOSI: now reaches Arduino1.14 (D11)
- net MOSI: now also Display1.4 (Pin_4)
- net LED: now reaches Arduino1.15 (D12)
- net LED: now also D1.2 (A)
- net CLK: now reaches Arduino1.16 (D13)
- net CLK: now also Display1.3 (Pin_3)
- net SW3: now reaches Arduino1.19 (A0)
- net SW3: now also R3.2, SW3.1
- net SW2: now reaches Arduino1.20 (A1)
- net SW2: now also R2.2, SW2.1
- net SW1: now reaches Arduino1.21 (A2)
- net SW1: now also R1.2, SW1.1
- net UART2_TX: now reaches Arduino1.22 (A3)
- net UART2_TX: now also UART2.3 (Pin_3)
- net UART2_RX: now reaches Arduino1.23 (A4)
- net UART2_RX: now also UART2.2 (Pin_2)
- net Analog1: now reaches Arduino1.24 (A5)
- net Analog1: now also An1.2 (Pin_2)
- net Analog2: now reaches Arduino1.25 (A6)
- net Analog2: now also An2.2 (Pin_2)
- net Analog3: now reaches Arduino1.26 (A7)
- net Analog3: now also An3.2 (Pin_2)
- net UART1_RX: now reaches Arduino1.5 (D2)
- net UART1_RX: now also UART1.2 (Pin_2)
- net UART1_TX: now reaches Arduino1.6 (D3)
- net UART1_TX: now also UART1.3 (Pin_3)
- net ARD_RX: now reaches Arduino1.7 (D4)
- net ARD_RX: now also GPS1.3 (Pin_3)
- net ARD_TX: now reaches Arduino1.8 (D5)
- net ARD_TX: now also GPS1.2 (Pin_2)
Other:
- moved on the sheet: Arduino1, Display1, Driver1, GPS1, Motor1, Power1
